Commit message: 1.add mid360 link

File: resources/elf2-ankle/urdf/elf2_ankle_dof12.urdf (robot description, URDF)
Before this commit: robot elf2, 28 links, 27 joints
Links:
- added link mid360_link
Joints:
- joint mid360_joint: child mid360 -> mid360_link; origin xyz=0 0 0.23988 rpy=3.1416 0 1.5708 -> xyz=0 0 0.2188 rpy=3.1416 0 1.5708

File: resources/elf2-ankle/urdf/elf2_ankle_dof25.urdf (robot description, URDF)
Before this commit: robot elf2, 28 links, 27 joints
Links:
- added link mid360_link
Joints:
- joint l_elb_y_joint: type fixed -> revolute
- joint l_elb_z_joint: type fixed -> revolute
- joint l_shld_x_joint: type fixed -> revolute
- joint l_shld_y_joint: type fixed -> revolute
- joint l_shld_z_joint: type fixed -> revolute
- joint mid360_joint: child mid360 -> mid360_link; origin xyz=0 0 0.23988 rpy=3.1416 0 1.5708 -> xyz=0 0 0.2188 rpy=3.1416 0 1.5708
- joint r_elb_y_joint: type fixed -> revolute
- joint r_elb_z_joint: type fixed -> revolute
- joint r_shld_x_joint: type fixed -> revolute
- joint r_shld_y_joint: type fixed -> revolute
- joint r_shld_z_joint: type fixed -> revolute
- joint waist_x_joint: type fixed -> revolute
- joint waist_y_joint: type fixed -> revolute
- joint waist_z_joint: type fixed -> revolute

File: resources/elf2-foot/urdf/elf2_foot_dof12.urdf (robot description, URDF)
Before this commit: robot elf2, 28 links, 27 joints
Links:
- added link mid360_link
Joints:
- joint l_elb_y_joint: type revolute -> fixed
- joint l_elb_z_joint: type revolute -> fixed
- joint l_shld_x_joint: type revolute -> fixed
- joint l_shld_y_joint: type revolute -> fixed
- joint l_shld_z_joint: type revolute -> fixed
- joint mid360_joint: child mid360 -> mid360_link; origin xyz=0 0 0.23988 rpy=3.1416 0 1.5708 -> xyz=0 0 0.2188 rpy=3.1416 0 1.5708
- joint r_elb_y_joint: type revolute -> fixed
- joint r_elb_z_joint: type revolute -> fixed
- joint r_shld_x_joint: type revolute -> fixed
- joint r_shld_y_joint: type revolute -> fixed
- joint r_shld_z_joint: type revolute -> fixed
- joint waist_x_joint: type revolute -> fixed
- joint waist_y_joint: type revolute -> fixed
- joint waist_z_joint: type revolute -> fixed

File: resources/elf2-trunk/urdf/elf2_trunk_dof25.urdf (robot description, URDF)
Before this commit: robot elf2, 28 links, 27 joints
Links:
- added link mid360_link
Joints:
- joint mid360_joint: child mid360 -> mid360_link; origin xyz=0 0 0.23988 rpy=3.1416 0 1.5708 -> xyz=0 0 0.2188 rpy=3.1416 0 1.5708

Commit message: 1.update urdf

File: resources/elf2-ankle/urdf/elf2_ankle_dof12.urdf (robot description, URDF)
Before this commit: robot elf2, 29 links, 27 joints
Links:
- link l_ankle_x_link: geometry collision mesh filename=../meshes/foot-240.STL; visual mesh filename=../meshes/foot-240.STL
- link r_ankle_x_link: geometry collision mesh filename=../meshes/foot-240.STL; visual mesh filename=../meshes/foot-240.STL
Joints:
- joint l_ankle_x_joint: limit lower=-0.349 upper=0.349 effort=6 velocity=20 -> lower=-0.349 upper=0.349 effort=20 velocity=20
- joint l_ankle_y_joint: limit lower=-2 upper=2 effort=12 velocity=20 -> lower=-2 upper=2 effort=50 velocity=20
- joint r_ankle_x_joint: limit lower=-0.349 upper=0.349 effort=6 velocity=20 -> lower=-0.349 upper=0.349 effort=20 velocity=20
- joint r_ankle_y_joint: limit lower=-2 upper=2 effort=12 velocity=20 -> lower=-2 upper=2 effort=50 velocity=20

File: resources/elf2-ankle/urdf/elf2_ankle_dof25.urdf (robot description, URDF)
Before this commit: robot elf2, 29 links, 27 joints
Links:
- link l_ankle_x_link: geometry collision mesh filename=../meshes/foot-240.STL; visual mesh filename=../meshes/foot-240.STL
- link r_ankle_x_link: geometry collision mesh filename=../meshes/foot-240.STL; visual mesh filename=../meshes/foot-240.STL
Joints:
- joint l_ankle_x_joint: limit lower=-0.349 upper=0.349 effort=6 velocity=20 -> lower=-0.349 upper=0.349 effort=20 velocity=20
- joint l_ankle_y_joint: limit lower=-2 upper=2 effort=12 velocity=20 -> lower=-2 upper=2 effort=50 velocity=20
- joint r_ankle_x_joint: limit lower=-0.349 upper=0.349 effort=6 velocity=20 -> lower=-0.349 upper=0.349 effort=20 velocity=20
- joint r_ankle_y_joint: limit lower=-2 upper=2 effort=12 velocity=20 -> lower=-2 upper=2 effort=50 velocity=20

File: resources/elf2-foot/urdf/elf2_foot_dof12.urdf (robot description, URDF)
Before this commit: robot elf2, 29 links, 27 joints
Links:
- link l_ankle_x_link: geometry collision mesh filename=../meshes/l_hum_foot.STL; visual mesh filename=../meshes/l_hum_foot.STL
- link r_ankle_x_link: geometry collision mesh filename=../meshes/r_hum_foot.STL; visual mesh filename=../meshes/r_hum_foot.STL
Joints:
- joint l_ankle_x_joint: limit lower=-0.349 upper=0.349 effort=6 velocity=20 -> lower=-0.349 upper=0.349 effort=20 velocity=20
- joint l_ankle_y_joint: limit lower=-2 upper=2 effort=12 velocity=20 -> lower=-2 upper=2 effort=50 velocity=20
- joint r_ankle_x_joint: limit lower=-0.349 upper=0.349 effort=6 velocity=20 -> lower=-0.349 upper=0.349 effort=20 velocity=20
- joint r_ankle_y_joint: limit lower=-2 upper=2 effort=12 velocity=20 -> lower=-2 upper=2 effort=50 velocity=20

File: resources/elf2-foot/urdf/elf2_foot_dof25.urdf (robot description, URDF)
Before this commit: robot elf2, 28 links, 27 joints
Links:
- link l_ankle_x_link: geometry collision mesh filename=../meshes/l_hum_foot.STL; visual mesh filename=../meshes/l_hum_foot.STL
- link r_ankle_x_link: geometry collision mesh filename=../meshes/r_hum_foot.STL; visual mesh filename=../meshes/r_hum_foot.STL
Joints:
- joint l_ankle_x_joint: limit lower=-0.349 upper=0.349 effort=6 velocity=20 -> lower=-0.349 upper=0.349 effort=20 velocity=20
- joint l_ankle_y_joint: limit lower=-2 upper=2 effort=12 velocity=20 -> lower=-2 upper=2 effort=50 velocity=20
- joint r_ankle_x_joint: limit lower=-0.349 upper=0.349 effort=6 velocity=20 -> lower=-0.349 upper=0.349 effort=20 velocity=20
- joint r_ankle_y_joint: limit lower=-2 upper=2 effort=12 velocity=20 -> lower=-2 upper=2 effort=50 velocity=20
