Commit message: update simulation add new dance
Co-authored-by: Copilot <copilot@github.com>

File: resources/elf3_dof29/urdf/elf3.urdf (robot description, URDF)
Before this commit: robot elf3, 36 links, 35 joints
Links:
- removed link neck_y_link
- removed link neck_z_link
- added link head_y_link, mass 1.57425673; collision mesh filename=./meshes/head_y_link.STL; visual mesh filename=./meshes/head_y_link.STL
- added link head_z_link, mass 0.37665142; collision mesh filename=./meshes/head_z_link.STL; visual mesh filename=./meshes/head_z_link.STL
Joints:
- removed joint neck_y_joint
- removed joint neck_z_joint
- added joint head_y_joint: type fixed, parent head_z_link, child head_y_link, origin xyz=0 0 0 rpy=0 0 0, axis 0 1 0, limit lower=-0.785 upper=0.785 effort=21 velocity=20
- added joint head_z_joint: type fixed, parent torso_link, child head_z_link, origin xyz=0 0 0.2995 rpy=0 0 0, axis 0 0 1, limit lower=-1.57 upper=1.57 effort=21 velocity=20
- joint d435i_joint: parent neck_y_link -> head_y_link
- joint mid360_joint: parent neck_y_link -> head_y_link

File: resources/elf3_dof29_hand/urdf/elf3.urdf (robot description, URDF)
Before this commit: robot elf3, 36 links, 35 joints
Links:
- removed link neck_y_link
- removed link neck_z_link
- added link head_y_link, mass 1.57425673; collision mesh filename=./meshes/head_y_link.STL; visual mesh filename=./meshes/head_y_link.STL
- added link head_z_link, mass 0.37665142; collision mesh filename=./meshes/head_z_link.STL; visual mesh filename=./meshes/head_z_link.STL
Joints:
- removed joint neck_y_joint
- removed joint neck_z_joint
- added joint head_y_joint: type fixed, parent head_z_link, child head_y_link, origin xyz=0 0 0 rpy=0 0 0, axis 0 1 0, limit lower=-0.785 upper=0.785 effort=21 velocity=20
- added joint head_z_joint: type fixed, parent torso_link, child head_z_link, origin xyz=0 0 0.2995 rpy=0 0 0, axis 0 0 1, limit lower=-1.57 upper=1.57 effort=21 velocity=20
- joint d435i_joint: parent neck_y_link -> head_y_link
- joint mid360_joint: parent neck_y_link -> head_y_link

File: resources/elf3_dof31_hand/urdf/elf3.urdf (robot description, URDF)
Before this commit: robot elf3, 36 links, 35 joints
Links:
- removed link neck_y_link
- removed link neck_z_link
- added link head_y_link, mass 1.57425673; collision mesh filename=./meshes/head_y_link.STL; visual mesh filename=./meshes/head_y_link.STL
- added link head_z_link, mass 0.37665142; collision mesh filename=./meshes/head_z_link.STL; visual mesh filename=./meshes/head_z_link.STL
Joints:
- removed joint neck_y_joint
- removed joint neck_z_joint
- added joint head_y_joint: type revolute, parent head_z_link, child head_y_link, origin xyz=0 0 0 rpy=0 0 0, axis 0 1 0, limit lower=-0.785 upper=0.785 effort=21 velocity=20
- added joint head_z_joint: type revolute, parent torso_link, child head_z_link, origin xyz=0 0 0.2995 rpy=0 0 0, axis 0 0 1, limit lower=-1.57 upper=1.57 effort=21 velocity=20
- joint d435i_joint: parent neck_y_link -> head_y_link
- joint mid360_joint: parent neck_y_link -> head_y_link
